Commit message: Imported upstream version '0.2.3' of 'upstream'

File: heron_description/urdf/accessories.urdf.xacro (robot description, xacro)
@@ -60,4 +60,13 @@
     </joint>
   </xacro:if>
+  <xacro:if value="$(optenv HERON_SONAR 0)">
+    <link name="sonar_$(optenv HERON_SONAR_MOUNT surface)" />
+    <joint name="$(optenv HERON_SONAR_MOUNT rear)_sonar_joint" type="fixed">
+    <origin xyz="$(optenv HERON_SONAR_OFFSET 0.0 0 -0.10)"
+            rpy="$(optenv HERON_SONAR_RPY 0 0 0)" />
+      <parent link="base_link" />
+      <child link="sonar_$(optenv HERON_SONAR_MOUNT surface)" />
+    </joint>
+  </xacro:if>
   <xacro:unless value="$(optenv HERON_LASER 0)">
     <rear_plate type="plain" />
