Commit message: Imported upstream version '0.3.0' of 'upstream'

File: heron_description/urdf/heron.urdf.xacro (robot description, xacro)
@@ -25,5 +25,5 @@
 This program contains the description of the robot base model for the Clearpath Heron
 -->
-<robot name="heron" xmlns:xacro="http://ros.org/wiki/xacro">
+<robot name="heron" xmlns:xacro="http://www.ros.org/wiki/xacro">
     <xacro:property name="PI" value="3.1415926535897931" />
     <xacro:property name="dummy_inertia" value="1e-09"/>
@@ -103,6 +103,6 @@
       <parent link="base_link" />
       <child link="imu_link" />
-      <origin xyz="$(optenv HERON_IMU_UM6_XYZ 0.015 0.0 0.072)"
-              rpy="$(optenv HERON_IMU_UM6_RPY 0.0 3.14159 1.5708)" />
+      <origin xyz="$(optenv HERON_IMU_UM6_XYZ -0.290 0.0 0.024)"
+              rpy="$(optenv HERON_IMU_UM6_RPY 3.14159 0.0 0.0)" />
     </joint>
     <link name="navsat_link" />
@@ -110,5 +110,5 @@
       <parent link="base_link" />
       <child link="navsat_link" />
-      <origin xyz="$(optenv HERON_NAVSAT_UBLOX_XYZ 0.015 -0.050 0.072)"
+      <origin xyz="$(optenv HERON_NAVSAT_UBLOX_XYZ 0.015 0.050 0.072)"
               rpy="$(optenv HERON_NAVSAT_UBLOX_RPY 0.0 0.0 0.0)" />
     </joint>
